File: power.kicad_sch (KiCad schematic)
At the start: 6 parts, among them J501 power, U501 Buck

Commit message: added something to debug the channel buttons
Parts:
- D501, D502: footprint Diode_THT:D_DO-34_SOD68_P7.62mm_Horizontal -> Diode_SMD:D_1206_3216Metric
Changed lines of the file:
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@@
     (property "Reference" "D501" (id 0) (at 128.27 64.8802 0))
     (property "Value" "D" (id 1) (at 128.27 67.4171 0))
-    (property "Footprint" "Diode_THT:D_DO-34_SOD68_P7.62mm_Horizontal" (id 2) (at 128.27 69.85 0)
+    (property "Footprint" "Diode_SMD:D_1206_3216Metric" (id 2) (at 128.27 69.85 0)
       (effects (font (size 1.27 1.27)) hide)
     )
@@
     (property "Reference" "D502" (id 0) (at 170.18 64.8802 0))
     (property "Value" "D" (id 1) (at 170.18 67.4171 0))
-    (property "Footprint" "Diode_THT:D_DO-34_SOD68_P7.62mm_Horizontal" (id 2) (at 170.18 69.85 0)
+    (property "Footprint" "Diode_SMD:D_1206_3216Metric" (id 2) (at 170.18 69.85 0)
       (effects (font (size 1.27 1.27)) hide)
     )
