File: mosfetAddon/mosfetAddon.kicad_sch (KiCad schematic)
At the start: 66 parts, among them J1 coil, J10 Conn_01x18_Male, J2 coil, J3 coil, J4 coil, J5 coil, J6 coil, J7 coil, J8 coil, J9 pow, Q1 FDS6890A, Q2 FDS6890A, Q3 FDS6890A, Q4 FDS6890A, Q5 FDS6890A, Q6 FDS6890A, Q7 FDS6890A, Q8 FDS6890A

Commit message: about to make new branch for control panel usage
Parts:
- removed Q1, Q2, Q3, Q4, Q5, Q6, Q7, Q8: FDS6890A, Package_SO:SOIC-8_3.9x4.9mm_P1.27mm, symbol Transistor_FET:FDS6890A
- added D17: (no value), symbol Device:D_Bridge_+-AA
- added Q1: (no value), symbol Transistor_FET:AO3400A
- added Q10, Q11, Q12, Q13, Q14, Q15, Q16, Q2, Q3, Q4, Q5, Q6, Q7, Q8, Q9: AO3400A, Package_TO_SOT_SMD:SOT-23, symbol Transistor_FET:AO3400A
- D1, D10, D11, D12, D13, D14, D15, D16, D2, D3, D4, D5, D6, D7, D8, D9: JLCPCB Part# (none) -> C8678
- R1, R10, R11, R12, R13, R14, R15, R16, R3, R4, R5, R6, R7, R8, R9: JLCPCB Part# (none) -> C17958
- R2: value 22R -> (none); footprint Resistor_SMD:R_1206_3216Metric_Pad1.30x1.75mm_HandSolder -> (none); JLCPCB Part# (none) -> C17958
- R201, R202, R203, R204, R205, R206, R207, R208, R209, R210, R211, R212, R213, R214, R215, R216: value 10k -> (none); footprint Resistor_SMD:R_1206_3216Metric_Pad1.30x1.75mm_HandSolder -> (none); JLCPCB Part# (none) -> C17902
Connections:
- net GND: now also D17.2 (-), Q1.2 (S), Q10.2 (S), Q11.2 (S), Q12.2 (S), Q13.2 (S), Q14.2 (S), Q15.2 (S), Q16.2 (S), Q2.2 (S), Q3.2 (S), Q4.2 (S), Q5.2 (S), Q6.2 (S), Q7.2 (S), Q8.2 (S), Q9.2 (S); no longer J9.1 (Pin_1)
- net coil1L: now also Q1.3 (D)
- net coil1R: now also Q2.3 (D)
- net coil2L: now also Q3.3 (D)
- net coil2R: now also Q4.3 (D)
- net coil3L: now also Q5.3 (D)
- net coil3R: now also Q6.3 (D)
- net coil4L: now also Q7.3 (D)
- net coil4R: now also Q8.3 (D)
- net coil5L: now also Q9.3 (D)
- net coil5R: now also Q10.3 (D)
- net coil6L: now also Q11.3 (D)
- net coil6R: now also Q12.3 (D)
- net coil7L: now also Q13.3 (D)
- net coil7R: now also Q14.3 (D)
- net coil8L: now also Q15.3 (D)
- net coil8R: now also Q16.3 (D)
- net pow: now also D17.1 (+); no longer J9.2 (Pin_2)
- net at R1.2, R201.2: now also Q2.1 (G)
- net at R16.2, R216.2: now also Q15.1 (G)
- net at R2.2, R202.2: now also Q1.1 (G)
- net at R14.2, R214.2: now also Q13.1 (G)
- net at R12.2, R212.2: now also Q11.1 (G)
- net at R205.2, R5.2: now also Q6.1 (G)
- net at R203.2, R3.2: now also Q4.1 (G)
- net at R204.2, R4.2: now also Q3.1 (G)
- net at R13.2, R213.2: now also Q14.1 (G)
- net at R15.2, R215.2: now also Q16.1 (G)
- net at R209.2, R9.2: now also Q10.1 (G)
- net at R208.2, R8.2: now also Q7.1 (G)
- net at R11.2, R211.2: now also Q12.1 (G)
- net at R207.2, R7.2: now also Q8.1 (G)
- net at R10.2, R210.2: now also Q9.1 (G)
- net at R206.2, R6.2: now also Q5.1 (G)
- new net: D17.3, J9.1 (Pin_1)
- new net: D17.4, J9.2 (Pin_2)
Other:
- moved on the sheet: J1, J3, J5, J7, J9
