File: currentSensor/currentSensor.kicad_sch (KiCad schematic)
At the start: 54 parts, among them J1 Conn_01x09_Male, J2 Conn_01x09_Male, J3 Screw_Terminal_01x08, J4 Screw_Terminal_01x02, J5 Screw_Terminal_01x08, U1 PC847, U2 PC847, U3 PC847, U4 PC847

Commit message: added some changed to the current sensor. There also seems a bug with the mcp23017. I suspect the chip itself may be damaged. Not all pins are at 5V
Parts:
- D1, D10, D11, D12, D13, D14, D15, D16, D2, D3, D4, D5, D6, D7, D8, D9: footprint Diode_THT:Diode_Bridge_DIP-4_W7.62mm_P5.08mm -> (none)
- R1, R10, R11, R12, R13, R14, R15, R16, R17, R18, R19, R2, R20, R21, R22, R23, R24, R25, R26, R27, R28, R29, R3, R4, R5, R6, R7, R8, R9: footprint Resistor_THT:R_Axial_DIN0204_L3.6mm_D1.6mm_P7.62mm_Horizontal -> (none)

Commit message: about to make new branch for control panel usage
Parts:
- added JP? (x4): Jumper_2_Bridged, symbol Jumper:Jumper_2_Bridged
- added JP? (x7): Jumper_2_Open, symbol Jumper:Jumper_2_Open
- added JP?: (no value), symbol Jumper:Jumper_2_Open
- added R? (x3): 1M, symbol Device:R
- added R? (x2): (no value), symbol Device:R
- added R? (x3): 20k, symbol Device:R
- D1, D10, D11, D12, D13, D14, D15, D16, D2, D3, D4, D5, D6, D7, D8, D9: footprint (none) -> Diode_SMD:Diode_Bridge_Diotec_SO-DIL-Slim
- R1, R10, R11, R12, R13, R14, R15, R16, R17, R18, R19, R2, R20, R21, R22, R23, R24, R25, R26, R27, R28, R29, R3, R4, R5, R6, R7, R8, R9: footprint (none) -> Resistor_SMD:R_1206_3216Metric
Connections:
- net GND: now also JP?.1 (A), JP?.1 (A), JP?.1 (A), JP?.1 (A)
- new net: JP?.1 (A), JP?.2 (B), R?.2, R?.2 (x4)
- new net: JP?.1 (A), R?.1 (x3)
- new net +5V: JP?.2 (B), JP?.2 (B), JP?.2 (B), JP?.2 (B), JP?.2 (B), JP?.2 (B), JP?.2 (B), JP?.2 (B)
Other:
- note added: "1 IO pin"

Commit message: added separate HAL files for NX and empty files for the MCP23017. They need filling in for read and write registers
Parts:
- removed D1, D10, D11, D12, D13, D14, D15, D16, D2, D3, D4, D5, D6, D7, D8, D9: D, Diode_SMD:Diode_Bridge_Diotec_SO-DIL-Slim, symbol Device:D_Bridge_+-AA
- removed J1, J2: Conn_01x09_Male, Connector_PinHeader_2.54mm:PinHeader_1x09_P2.54mm_Horizontal, symbol Connector:Conn_01x09_Male
- removed JP? (x4): Jumper_2_Bridged, symbol Jumper:Jumper_2_Bridged
- removed JP? (x7): Jumper_2_Open, symbol Jumper:Jumper_2_Open
- removed JP?: (no value), symbol Jumper:Jumper_2_Open
- removed R? (x3): 1M, symbol Device:R
- removed R? (x2): (no value), symbol Device:R
- removed R? (x3): 20k, symbol Device:R
- removed U1, U2, U3, U4: PC847, Package_DIP:DIP-16_W7.62mm, symbol Isolator:PC847
- added D1, D10, D11, D12, D13, D14, D15, D16, D2, D3, D4, D5, D6, D7, D8, D9: ABS2, Diode_SMD:Diode_Bridge_Diotec_ABS, symbol Diode_Bridge:ABS2
- added J4, J5: Conn_01x10_Male, Connector_PinHeader_2.54mm:PinHeader_1x10_P2.54mm_Horizontal, symbol Connector:Conn_01x10_Male
- added R30, R32: 4k7, Resistor_SMD:R_0805_2012Metric_Pad1.20x1.40mm_HandSolder, symbol Device:R
- added R31: 47R, Resistor_SMD:R_0805_2012Metric_Pad1.20x1.40mm_HandSolder, symbol Device:R
- added U1, U10, U11, U12, U13, U14, U15, U16, U2, U3, U4, U5, U6, U7, U8, U9: SFH6206-2T, Package_DIP:SMDIP-4_W9.53mm_Clearance8mm, symbol Isolator:SFH6206-2T
- R1, R11, R13, R15, R17, R19, R21, R23, R25, R27, R29, R3, R5, R7, R9: value R -> 47R; footprint Resistor_SMD:R_1206_3216Metric -> Resistor_SMD:R_0805_2012Metric_Pad1.20x1.40mm_HandSolder; JLCPCB Part# (none) -> C17714
- R10, R12, R14, R16, R18, R2, R20, R22, R24, R26, R28, R4, R6, R8: value R -> 4k7; footprint Resistor_SMD:R_1206_3216Metric -> Resistor_SMD:R_0805_2012Metric_Pad1.20x1.40mm_HandSolder; JLCPCB Part# (none) -> C17673
- renumbered J3 to J1, J4 to J2, J5 to J3
Connections:
- net +5V: now also J4.1 (Pin_1), J5.1 (Pin_1)
- net COM: now also R10.2, R12.2, R14.2, R16.2, R2.2, R4.2, R6.2, R8.2, D1.4, D10.4, D11.4, D12.4, D13.4, D14.4, D15.4, D16.4, D2.4, D3.4, D4.4, D5.4, D6.4, D7.4, D8.4, D9.4, R30.2, R32.2, U1.2, U10.2, U11.2, U12.2, U13.2, U14.2, U15.2, U16.2, U2.2, U3.2, U4.2, U5.2, U6.2, U7.2, U8.2, U9.2; no longer R17.2, R19.2, R21.2, R23.2, R25.2, R27.2, R29.2
- net GND: now also J4.10 (Pin_10), J5.10 (Pin_10), U1.3, U10.3, U11.3, U12.3, U13.3, U14.3, U15.3, U16.3, U2.3, U3.3, U4.3, U5.3, U6.3, U7.3, U8.3, U9.3
- net inp1: now also J4.2 (Pin_2), U1.4
- net inp10: now also J5.3 (Pin_3), U10.4
- net inp11: now also J5.4 (Pin_4), U11.4
- net inp12: now also J5.5 (Pin_5), U12.4
- net inp13: now also J5.6 (Pin_6), U13.4
- net inp14: now also J5.7 (Pin_7), U14.4
- net inp15: now also J5.8 (Pin_8), U15.4
- net inp16: now also J5.9 (Pin_9), U16.4
- net inp2: now also J4.3 (Pin_3), U2.4
- net inp3: now also J4.4 (Pin_4), U3.4
- net inp4: now also J4.5 (Pin_5), U4.4
- net inp5: now also J4.6 (Pin_6), U5.4
- net inp6: now also J4.7 (Pin_7), U6.4
- net inp7: now also J4.8 (Pin_8), U7.4
- net inp8: now also J4.9 (Pin_9), U8.4
- net inp9: now also J5.2 (Pin_2), U9.4
- net track1: now also J1.8 (Pin_8), R1.1, R2.1, D1.3; no longer J1.1 (Pin_1), R21.1, R5.1
- net track10: now also J3.7 (Pin_7), R19.1, R20.1, D10.3; no longer J3.2 (Pin_2), R10.1, R26.1
- net track11: now also J3.6 (Pin_6), R21.1, R22.1, D11.3; no longer J3.3 (Pin_3), R11.1, R27.1
- net track12: now also J3.5 (Pin_5), R23.1, R24.1, D12.3; no longer J3.4 (Pin_4), R12.1, R28.1
- net track13: now also J3.4 (Pin_4), R25.1, R26.1, D13.3; no longer J3.5 (Pin_5), R13.1, R29.1
- net track14: now also J3.3 (Pin_3), R27.1, R28.1, D14.3; no longer J3.6 (Pin_6), R14.1
- net track15: now also J3.2 (Pin_2), R29.1, D15.3, R30.1; no longer J3.7 (Pin_7), R15.1
- net track16: now also J3.1 (Pin_1), D16.3, R31.1, R32.1; no longer J3.8 (Pin_8), R16.1
- net track2: now also J1.7 (Pin_7), R3.1, R4.1, D2.3; no longer J1.2 (Pin_2), R22.1, R6.1
- net track3: now also J1.6 (Pin_6), R5.1, R6.1, D3.3; no longer J1.3 (Pin_3), R23.1, R7.1
- net track4: now also J1.5 (Pin_5), R7.1, D4.3; no longer J1.4 (Pin_4), R24.1
- net track5: now also J1.4 (Pin_4), R10.1, R9.1, D5.3; no longer J1.5 (Pin_5), R1.1, R17.1
- net track6: now also J1.3 (Pin_3), R11.1, R12.1, D6.3; no longer J1.6 (Pin_6), R18.1, R2.1
- net track7: now also J1.2 (Pin_2), R13.1, R14.1, D7.3; no longer J1.7 (Pin_7), R19.1, R3.1
- net track8: now also J1.1 (Pin_1), R15.1, R16.1, D8.3; no longer J1.8 (Pin_8), R20.1, R4.1
- net track9: now also J3.8 (Pin_8), R17.1, R18.1, D9.3; no longer J3.1 (Pin_1), R25.1, R9.1
- net at R13.2: now also U7.1
- net at R5.2: now also U3.1
- net at R15.2: now also U8.1
- net at R1.2: now also U1.1
- net at R9.2: now also U5.1
- net at R7.2: now also U4.1
- net at R3.2: now also U2.1
- net at R11.2: now also U6.1
- new net: D6.1 (+), D6.2 (-)
- new net: D14.1 (+), D14.2 (-)
- new net: D2.1 (+), D2.2 (-)
- new net: R25.2, U13.1
- new net: R27.2, U14.1
- new net: D8.1 (+), D8.2 (-)
- new net: D3.1 (+), D3.2 (-)
- new net: R21.2, U11.1
- new net: D5.1 (+), D5.2 (-)
- new net: R19.2, U10.1
- new net: D7.1 (+), D7.2 (-)
- new net: D13.1 (+), D13.2 (-)
- new net: R23.2, U12.1
- new net: D15.1 (+), D15.2 (-)
- new net: R17.2, U9.1
- new net: D4.1 (+), D4.2 (-)
- new net: R31.2, U16.1
- new net: D12.1 (+), D12.2 (-)
- new net: D11.1 (+), D11.2 (-)
- new net: R29.2, U15.1
- new net: D9.1 (+), D9.2 (-)
- new net: D16.1 (+), D16.2 (-)
- new net: D10.1 (+), D10.2 (-)
- new net: D1.1 (+), D1.2 (-)
Other:
- note removed: "1 IO pin"
